File: kiCad Files/TransmitterCircuit/TransmitterLaser/TransmitterLaser.kicad_sch (KiCad schematic)
At the start: 15 parts, among them SW1 SW_SPDT, SW2 SW_SPDT, U1 74LS73, U2 74LS02

Commit message: creds to schematic
Parts:
- R1: value 1k -> 100
- R2: value 1.5k -> 120
Other:
- note added: "By Rosnel Leyva"
- note added: "Transmitter Circuit"
Changed lines of the file:
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@@
     (stroke (width 0) (type default) (color 0 0 0 0))
   )
+  (text "Transmitter Circuit\n" (at 186.563 190.627 0)
+    (effects (font (size 1.27 1.27)) (justify left bottom))
+  )
   (text "LOGIC FOR AMMO FUNC.\n" (at 206.375 19.558 0)
+    (effects (font (size 1.27 1.27)) (justify left bottom))
+  )
+  (text "By Rosnel Leyva\n" (at 216.662 186.563 0)
     (effects (font (size 1.27 1.27)) (justify left bottom))
   )
@@
       (effects (font (size 1.27 1.27)) (justify left))
     )
-    (property "Value" "1.5k" (id 1) (at 58.039 72.5169 0)
+    (property "Value" "120" (id 1) (at 58.039 72.5169 0)
       (effects (font (size 1.27 1.27)) (justify left))
     )
@@
       (effects (font (size 1.27 1.27)) (justify left))
     )
-    (property "Value" "1k" (id 1) (at 57.658 52.1969 0)
+    (property "Value" "100" (id 1) (at 57.658 52.1969 0)
       (effects (font (size 1.27 1.27)) (justify left))
     )
@@
     )
     (path "/ab081c8c-de9b-4711-b73f-6f39b550b93d"
-      (reference "R1") (unit 1) (value "1k") (footprint "Resistor_THT:R_Axial_DIN0204_L3.6mm_D1.6mm_P7.62mm_Horizontal")
+      (reference "R1") (unit 1) (value "100") (footprint "Resistor_THT:R_Axial_DIN0204_L3.6mm_D1.6mm_P7.62mm_Horizontal")
     )
     (path "/36ff31bc-7434-4f81-a2ef-85ae94f95350"
-      (reference "R2") (unit 1) (value "1.5k") (footprint "Resistor_THT:R_Axial_DIN0204_L3.6mm_D1.6mm_P7.62mm_Horizontal")
+      (reference "R2") (unit 1) (value "120") (footprint "Resistor_THT:R_Axial_DIN0204_L3.6mm_D1.6mm_P7.62mm_Horizontal")
     )
     (path "/5f24295e-d28f-4bf9-93d8-42f452b10d7f"
